File: gse2-hardware.kicad_pcb (KiCad board)
At the start: 2 copper layers, 3.2 x 15.6 mm, 300 parts, among them J1 PJ-002A, J10 Solenoid, J11 Solenoid, J12 Solenoid, J13 Solenoid, J14 E-MATCH, J15 E-MATCH, J16 ARM, J17 ALARM, J18 PT, J19 PT, J2 PJ-002A, J20 PT, J21 PT, J22 PT, J23 PT, J24 PT, J25 PT, J26 PT, J27 PT, J28 PT, J29 PT, J3 ARM Cortex Debug, J30 PT, J31 PT, J32 PT, J35 PT, J4 USB-C, J5 Solenoid, J6 Solenoid, J7 Solenoid, J8 Solenoid, J9 Solenoid, Q1 DMP3099L, Q10 DMG3402L, Q11 DMG3402L, Q12 DMG3402L, Q13 DMG3402L, Q14 DMG3402L, Q15 DMG3402L, Q2 DMG3402L, Q3 DMG3402L, Q4 DMG3402L, Q5 DMG3402L, Q6 DMG3402L, Q7 DMG3402L, Q8 DMG3402L, Q9 DMG3402L, U27 USBLC6-2SC6, Y1 16MHz

Commit message: Updated to add beginnings of layout. Most major subsystems internally layed out
Parts:
- removed C56: 10uF, Capacitor_SMD:C_0603_1608Metric
- removed J35: PT, 0UCIRP-KiCAD-Lib:GX-12 3 pin
- removed L2, L3: 3.3uH, Inductor_SMD:L_0603_1608Metric
- removed R2: 100K, Resistor_SMD:R_0402_1005Metric
- removed U33: ~, Package_TO_SOT_SMD:SOT-23-5
- added C101: 100nF, Capacitor_SMD:C_0402_1005Metric, F.Cu at (141.9, 132.6)
- added C102: ?, Capacitor_SMD:C_0402_1005Metric, F.Cu at (141.9, 134.6)
- added C103: 100nF, Capacitor_SMD:C_0402_1005Metric, F.Cu at (141.9, 136.5)
- added C104: 100nF, Capacitor_SMD:C_0402_1005Metric, F.Cu at (121.6, 132.6)
- added C105: ?, Capacitor_SMD:C_0402_1005Metric, F.Cu at (121.6, 134.6)
- added C106: 100nF, Capacitor_SMD:C_0402_1005Metric, F.Cu at (121.6, 136.5)
- added C107: 100nF, Capacitor_SMD:C_0402_1005Metric, F.Cu at (141.9, 151.7)
- added C108: ?, Capacitor_SMD:C_0402_1005Metric, F.Cu at (141.9, 153.7)
- added C109: 100nF, Capacitor_SMD:C_0402_1005Metric, F.Cu at (141.9, 155.6)
- added C60: 100nF, Capacitor_SMD:C_0402_1005Metric, F.Cu at (121.6, 155.6)
- added C69: ?, Capacitor_SMD:C_0402_1005Metric, B.Cu at (30.3, 94.9)
- added C70: ?, Capacitor_SMD:C_0402_1005Metric, B.Cu at (71.1, 111.1)
- added C71: ?, Capacitor_SMD:C_0402_1005Metric, B.Cu at (30.6, 132.2)
- added C72: ?, Capacitor_SMD:C_0402_1005Metric, B.Cu at (91.3, 132.2)
- added C73: ?, Capacitor_SMD:C_0402_1005Metric, B.Cu at (50.8, 111.1)
- added C74: ?, Capacitor_SMD:C_0402_1005Metric, B.Cu at (71.1, 153.3)
- added C75: ?, Capacitor_SMD:C_0402_1005Metric, B.Cu at (50.8, 132.2)
- added C76: ?, Capacitor_SMD:C_0402_1005Metric, B.Cu at (50.8, 153.3)
- added C77: ?, Capacitor_SMD:C_0402_1005Metric, B.Cu at (30.6, 111.1)
- added C78: ?, Capacitor_SMD:C_0402_1005Metric, B.Cu at (71.1, 132.2)
- added C79: ?, Capacitor_SMD:C_0402_1005Metric, B.Cu at (30.6, 153.3)
- added C80: ?, Capacitor_SMD:C_0402_1005Metric, B.Cu at (91.3, 111.1)
- added C81: ?, Capacitor_SMD:C_0402_1005Metric, F.Cu at (111.4, 117.4)
- added C82: ?, Capacitor_SMD:C_0402_1005Metric, F.Cu at (133.1, 97.0)
- added C83: ?, Capacitor_SMD:C_0402_1005Metric, F.Cu at (111.4, 96.3)
- added C84: 100nF, Capacitor_SMD:C_0402_1005Metric, F.Cu at (111.4, 119.3)
- added C85: 100nF, Capacitor_SMD:C_0402_1005Metric, F.Cu at (133.1, 99.0)
- added C86: 100nF, Capacitor_SMD:C_0402_1005Metric, F.Cu at (111.4, 98.3)
- added C87: 100nF, Capacitor_SMD:C_0402_1005Metric, B.Cu at (27.8, 99.2)
- added C88: 100nF, Capacitor_SMD:C_0402_1005Metric, B.Cu at (68.6, 115.4)
- added C89: 100nF, Capacitor_SMD:C_0402_1005Metric, B.Cu at (28.1, 136.5)
- added C90: 100nF, Capacitor_SMD:C_0402_1005Metric, B.Cu at (88.8, 136.5)
- added C91: 100nF, Capacitor_SMD:C_0402_1005Metric, B.Cu at (48.3, 115.4)
- added C92: 100nF, Capacitor_SMD:C_0402_1005Metric, B.Cu at (68.6, 157.5)
- added C93: 100nF, Capacitor_SMD:C_0402_1005Metric, B.Cu at (48.3, 136.5)
- added C94: 100nF, Capacitor_SMD:C_0402_1005Metric, B.Cu at (48.3, 157.5)
- added C95: 100nF, Capacitor_SMD:C_0402_1005Metric, B.Cu at (28.1, 115.4)
- added C96: 100nF, Capacitor_SMD:C_0402_1005Metric, B.Cu at (68.6, 136.5)
- added C97: 100nF, Capacitor_SMD:C_0402_1005Metric, B.Cu at (28.1, 157.5)
- added C98: 100nF, Capacitor_SMD:C_0402_1005Metric, B.Cu at (88.8, 115.4)
- added D26: BZT52H, Diode_SMD:D_SOD-123F, B.Cu at (27.3, 95.9)
- added D27: BZT52H, Diode_SMD:D_SOD-123F, B.Cu at (68.1, 112.1)
- added D28: BZT52H, Diode_SMD:D_SOD-123F, B.Cu at (27.6, 133.2)
- added D29: BZT52H, Diode_SMD:D_SOD-123F, B.Cu at (88.3, 133.2)
- added D30: BZT52H, Diode_SMD:D_SOD-123F, B.Cu at (47.8, 112.1)
- added D31: BZT52H, Diode_SMD:D_SOD-123F, B.Cu at (68.1, 154.3)
- added D32: BZT52H, Diode_SMD:D_SOD-123F, B.Cu at (47.8, 133.2)
- added D33: BZT52H, Diode_SMD:D_SOD-123F, B.Cu at (47.8, 154.3)
- added D34: BZT52H, Diode_SMD:D_SOD-123F, B.Cu at (27.6, 112.1)
- added D35: BZT52H, Diode_SMD:D_SOD-123F, B.Cu at (68.1, 133.2)
- added D36: BZT52H, Diode_SMD:D_SOD-123F, B.Cu at (27.6, 154.3)
- added D37: BZT52H, Diode_SMD:D_SOD-123F, B.Cu at (88.3, 112.1)
- added D38: BZT52C3V3LP-7, Diode_SMD:D_0402_1005Metric_Pad0.77x0.64mm_HandSolder, F.Cu at (114.7, 115.4)
- added D39: BZT52C3V3LP-7, Diode_SMD:D_0402_1005Metric_Pad0.77x0.64mm_HandSolder, F.Cu at (136.4, 95.0)
- added D40: BZT52C3V3LP-7, Diode_SMD:D_0402_1005Metric_Pad0.77x0.64mm_HandSolder, F.Cu at (114.7, 94.3)
- added D42: BZT52C3V3LP-7, Diode_SMD:D_0402_1005Metric_Pad0.77x0.64mm_HandSolder, F.Cu at (111.9, 155.5)
- added D43: BZT52C3V3LP-7, Diode_SMD:D_0402_1005Metric_Pad0.77x0.64mm_HandSolder, F.Cu at (132.1, 136.5)
- added D44: BZT52C3V3LP-7, Diode_SMD:D_0402_1005Metric_Pad0.77x0.64mm_HandSolder, F.Cu at (111.9, 136.5)
- added D45: BZT52C3V3LP-7, Diode_SMD:D_0402_1005Metric_Pad0.77x0.64mm_HandSolder, F.Cu at (132.1, 155.5)
- added J36: POT, 0UCIRP-KiCAD-Lib:GX-12 3 pin, F.Cu at (133.1, 131.4)
- added J37: POT, 0UCIRP-KiCAD-Lib:GX-12 3 pin, F.Cu at (113.7, 125.8)
- added J38: POT, 0UCIRP-KiCAD-Lib:GX-12 3 pin, F.Cu at (133.9, 144.9)
- added J39: Solenoid, 0UCIRP-KiCAD-Lib:GX-16 3 pin, F.Cu at (341.8, 20.4)
- added R108: 500R, Resistor_SMD:R_0402_1005Metric, F.Cu at (128.8, 136.5)
- added R118: 0R, Resistor_SMD:R_0402_1005Metric, B.Cu at (92.6, 132.2)
- added R119: 0R, Resistor_SMD:R_0402_1005Metric, B.Cu at (52.1, 111.1)
- added R120: 0R, Resistor_SMD:R_0402_1005Metric, B.Cu at (72.3, 153.3)
- added R121: 0R, Resistor_SMD:R_0402_1005Metric, B.Cu at (52.1, 132.2)
- added R122: 0R, Resistor_SMD:R_0402_1005Metric, B.Cu at (52.1, 153.3)
- added R123: 0R, Resistor_SMD:R_0402_1005Metric, B.Cu at (31.8, 111.1)
- added R124: 0R, Resistor_SMD:R_0402_1005Metric, B.Cu at (72.3, 132.2)
- added R125: 0R, Resistor_SMD:R_0402_1005Metric, B.Cu at (31.8, 153.3)
- added R126: 0R, Resistor_SMD:R_0402_1005Metric, B.Cu at (92.6, 111.1)
- added R127: 0R, Resistor_SMD:R_0402_1005Metric, F.Cu at (108.6, 119.4)
- added R128: 0R, Resistor_SMD:R_0402_1005Metric, F.Cu at (130.2, 99.0)
- added R129: 0R, Resistor_SMD:R_0402_1005Metric, F.Cu at (108.6, 98.3)
- added R131: 0R, Resistor_SMD:R_0402_1005Metric, F.Cu at (128.8, 138.5)
- added R132: 500R, Resistor_SMD:R_0402_1005Metric, F.Cu at (108.6, 136.5)
- added R133: 0R, Resistor_SMD:R_0402_1005Metric, F.Cu at (108.6, 138.5)
- added R134: 500R, Resistor_SMD:R_0402_1005Metric, F.Cu at (128.8, 155.5)
- added R135: 0R, Resistor_SMD:R_0402_1005Metric, F.Cu at (128.8, 157.5)
- added U35: ~, Package_TO_SOT_SMD:TO-252-2, B.Cu at (214.3, 120.3)
- added U36: ~, Package_TO_SOT_SMD:SOT-23-5, F.Cu at (122.8, 143.8)
- added U37: ~, Package_TO_SOT_SMD:SOT-23-5, F.Cu at (122.8, 148.5)
- added U38: ~, Package_TO_SOT_SMD:SOT-23-5, F.Cu at (143.0, 124.8)
- added U39: ~, Package_TO_SOT_SMD:SOT-23-5, B.Cu at (30.6, 98.2)
- added U40: ~, Package_TO_SOT_SMD:SOT-23-5, B.Cu at (71.3, 114.4)
- added U41: ~, Package_TO_SOT_SMD:SOT-23-5, B.Cu at (30.8, 135.5)
- added U42: ~, Package_TO_SOT_SMD:SOT-23-5, B.Cu at (91.6, 135.5)
- added U43: ~, Package_TO_SOT_SMD:SOT-23-5, B.Cu at (51.1, 114.4)
- added U44: ~, Package_TO_SOT_SMD:SOT-23-5, B.Cu at (71.3, 156.5)
- added U45: ~, Package_TO_SOT_SMD:SOT-23-5, B.Cu at (51.1, 135.5)
- added U46: ~, Package_TO_SOT_SMD:SOT-23-5, B.Cu at (51.1, 156.5)
- added U47: ~, Package_TO_SOT_SMD:SOT-23-5, B.Cu at (30.8, 114.4)
- added U48: ~, Package_TO_SOT_SMD:SOT-23-5, B.Cu at (71.3, 135.5)
- added U49: ~, Package_TO_SOT_SMD:SOT-23-5, B.Cu at (30.8, 156.5)
- added U50: ~, Package_TO_SOT_SMD:SOT-23-5, B.Cu at (91.6, 114.4)
- added U51: ~, Package_TO_SOT_SMD:SOT-23-5, F.Cu at (122.8, 108.3)
- added U52: ~, Package_TO_SOT_SMD:SOT-23-5, F.Cu at (144.5, 88.0)
- added U53: ~, Package_TO_SOT_SMD:SOT-23-5, F.Cu at (122.8, 87.3)
- added U55: ~, Package_TO_SOT_SMD:SOT-23-5, F.Cu at (143.0, 129.4)
- added U56: ~, Package_TO_SOT_SMD:SOT-23-5, F.Cu at (122.8, 124.8)
- added U57: ~, Package_TO_SOT_SMD:SOT-23-5, F.Cu at (122.8, 129.4)
- added U58: ~, Package_TO_SOT_SMD:SOT-23-5, F.Cu at (143.0, 143.8)
- added U59: ~, Package_TO_SOT_SMD:SOT-23-5, F.Cu at (143.0, 148.5)
- C11, C12, C13, C14, C16, C17, C18, C19, C20, C21, C28, C29, C30, C31, C34, C35, C36, C37, C38, C39, C40, C41, C45, C46, C47, C48, C57, D10, D11, D12, D13, D14, D15, D16, D17, D18, D19, D2, D20, D21, D22, D23, D24, D25, D8, D9, F1, L1, Q1, Q10, Q2, Q3, Q4, Q5, Q6, Q7, Q8, Q9, R1, R11, R13, R14, R17, R18, R19, R20, R21, R22, R23, R24, R25, R26, R27, R28, R29, R30, R31, R32, R33, R34, R35, R36, R37, R38, R39, R4, R40, R41, R42, R43, R44, R45, R46, R47, R48, R49, R67, R68, R70, R72, R74, R76, R78, R80, R84, R86, R88, R90, R92, R93, R94, R95, R96, R97, R98, R99, U1, U10, U11, U12, U15, U16, U17, U18, U20, U21, U22, U23, U24, U25, U26, U28, U29, U3, U30, U5, U6, U7, U8, U9: moved to B.Cu
- C42, C52: value 0.1uF -> 100nF; moved to B.Cu
- C43, C49, C54, C62: value 0.1uF -> 10nF; moved to B.Cu
- C50: value 100nF -> 0.33uF; footprint Capacitor_SMD:C_0603_1608Metric -> Capacitor_SMD:C_1206_3216Metric; moved to B.Cu
- C51: value 10uF -> 0.1uF; footprint Capacitor_SMD:C_0603_1608Metric -> Capacitor_SMD:C_1206_3216Metric; moved to B.Cu
- C55: footprint Capacitor_SMD:C_0603_1608Metric -> Capacitor_SMD:C_0402_1005Metric
- C59: value 100nF -> ?
- J18, J30, J31: value PT -> 420Sensor
- J32: value PT -> POT
- J9: value Solenoid -> PT; footprint 0UCIRP-KiCAD-Lib:GX-16 3 pin -> 0UCIRP-KiCAD-Lib:GX-12 3 pin
- R104: value 500R -> 0R; moved to B.Cu
- R105: value 165R -> 0R; moved to B.Cu
- R3: value 15K -> 500R
- R6: value 100K -> 0R
- R66, R69, R71, R73, R75, R77, R79, R81, R85, R87, R89, R91: value 10R -> 500R; moved to B.Cu
- R7: value 15K -> 0R; moved to B.Cu
- moved D9 273.7 mm to (354.2, 105.2)
- moved J13 273.1 mm to (348.7, 115.6)
- moved J8 273.0 mm to (344.8, 53.5)
- moved R14 270.8 mm to (352.7, 101.9), turned to 180 degrees
- moved D25 268.9 mm to (349.1, 40.1)
- moved R48 265.9 mm to (347.6, 36.8), turned to 180 degrees
- moved R11 264.0 mm to (354.2, 98.8), turned to 90 degrees
- moved R13 262.9 mm to (353.0, 98.8), turned to -90 degrees
- moved R17 260.0 mm to (350.2, 104.5)
- moved R46 259.1 mm to (349.1, 33.7), turned to 90 degrees
- moved C12 258.6 mm to (343.3, 104.8), turned to -90 degrees
- moved R47 258.0 mm to (347.9, 33.7), turned to -90 degrees
- moved Q2 256.6 mm to (350.6, 97.7), turned to 90 degrees
- moved D8 255.7 mm to (346.0, 99.4), turned to 90 degrees
- moved D11 255.1 mm to (324.6, 164.2)
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Connections:
- net /PT10_read renamed Net-(U28--)
- net /PT11_read renamed Net-(U29--)
- net /PT3_read renamed Net-(U18--)
- net /PT4_read renamed Net-(U20--)
- net /PT5_read renamed Net-(U21--)
- net /PT6_read renamed Net-(U22--)
- net /PT7_read renamed Net-(U23--)
- net /PT8_read renamed Net-(U24--)
- net /PT9_read renamed Net-(U25--)
- C28 pad 1: +3.3V -> +10V
- C29 pad 1: +3.3V -> +10V
- C30 pad 1: +3.3V -> +10V
- C31 pad 1: +3.3V -> +10V
- C34 pad 1: +3.3V -> +10V
- C35 pad 1: +3.3V -> +10V
- C36 pad 1: +3.3V -> +10V
- C37 pad 1: +3.3V -> +10V
- C38 pad 1: +3.3V -> +10V
- C39 pad 1: +3.3V -> +10V
- C40 pad 1: +3.3V -> +10V
- C41 pad 1: +3.3V -> +10V
- C43 pad 2: /NDQ_AI_GND -> GND
- C49 pad 2: /NDQ_AI_GND -> GND
- C50 pad 1: /LoadCell1/PWR -> GND
- C50 pad 2: GND -> +24V
- C51 pad 1: /LoadCell1/PWR -> +10V_LOAD_CELL
- C54 pad 1: /NDQ_AI_GND -> GND
- C55 pad 1: /LoadCell0/PWR -> +3.3V
- C59 pad 1: +3.3V -> Net-(U37-+)
- C62 pad 1: /NDQ_AI_GND -> GND
- GX-1 pad 2: /LoadCell0/PWR -> +10V_LOAD_CELL
- GX-2 pad 2: /LoadCell1/PWR -> +10V_LOAD_CELL
- J10 pad 2: Net-(D18-A) -> Net-(D16-A)
- J11 pad 2: Net-(D20-A) -> Net-(D18-A)
- J12 pad 2: Net-(D22-A) -> Net-(D20-A)
- J13 pad 2: Net-(D24-A) -> Net-(D22-A)
- J18 pad 2: Net-(J18-Pin_2) -> unconnected-(J18-Pin_2-Pad2)
- J18 pad 3: unconnected-(J18-Pin_3-Pad3) -> Net-(J18-Pin_3)
- J19 pad 2: Net-(J19-Pin_2) -> unconnected-(J19-Pin_2-Pad2)
- J19 pad 3: unconnected-(J19-Pin_3-Pad3) -> Net-(J19-Pin_3)
- J20 pad 2: Net-(J20-Pin_2) -> unconnected-(J20-Pin_2-Pad2)
- J20 pad 3: unconnected-(J20-Pin_3-Pad3) -> Net-(J20-Pin_3)
- J21 pad 2: Net-(J21-Pin_2) -> unconnected-(J21-Pin_2-Pad2)
- J21 pad 3: unconnected-(J21-Pin_3-Pad3) -> Net-(J21-Pin_3)
- J22 pad 2: Net-(J22-Pin_2) -> unconnected-(J22-Pin_2-Pad2)
- J22 pad 3: unconnected-(J22-Pin_3-Pad3) -> Net-(J22-Pin_3)
- J23 pad 2: Net-(J23-Pin_2) -> unconnected-(J23-Pin_2-Pad2)
- J23 pad 3: unconnected-(J23-Pin_3-Pad3) -> Net-(J23-Pin_3)
- J24 pad 2: Net-(J24-Pin_2) -> unconnected-(J24-Pin_2-Pad2)
- J24 pad 3: unconnected-(J24-Pin_3-Pad3) -> Net-(J24-Pin_3)
- J25 pad 2: Net-(J25-Pin_2) -> unconnected-(J25-Pin_2-Pad2)
- J25 pad 3: unconnected-(J25-Pin_3-Pad3) -> Net-(J25-Pin_3)
- J26 pad 2: Net-(J26-Pin_2) -> unconnected-(J26-Pin_2-Pad2)
- J26 pad 3: unconnected-(J26-Pin_3-Pad3) -> Net-(J26-Pin_3)
- J27 pad 2: Net-(J27-Pin_2) -> unconnected-(J27-Pin_2-Pad2)
- J27 pad 3: unconnected-(J27-Pin_3-Pad3) -> Net-(J27-Pin_3)
- J28 pad 2: Net-(J28-Pin_2) -> unconnected-(J28-Pin_2-Pad2)
- J28 pad 3: unconnected-(J28-Pin_3-Pad3) -> Net-(J28-Pin_3)
- J29 pad 2: Net-(J29-Pin_2) -> unconnected-(J29-Pin_2-Pad2)
- J29 pad 3: unconnected-(J29-Pin_3-Pad3) -> Net-(J29-Pin_3)
- J30 pad 2: Net-(J30-Pin_2) -> unconnected-(J30-Pin_2-Pad2)
- J30 pad 3: unconnected-(J30-Pin_3-Pad3) -> Net-(J30-Pin_3)
- J31 pad 2: Net-(J31-Pin_2) -> unconnected-(J31-Pin_2-Pad2)
- J31 pad 3: unconnected-(J31-Pin_3-Pad3) -> Net-(J31-Pin_3)
- J32 pad 1: +20V -> +3.3V
- J32 pad 3: unconnected-(J32-Pin_3-Pad3) -> GND
- J5 pad 2: Net-(D8-A) -> Net-(D10-A)
- J6 pad 2: Net-(D12-A) -> Net-(D8-A)
- J7 pad 2: Net-(D14-A) -> Net-(D12-A)
- J8 pad 2: Net-(D16-A) -> Net-(D14-A)
- J9 pad 1: +24V -> +20V
- J9 pad 2: Net-(D10-A) -> unconnected-(J9-Pin_2-Pad2)
- J9 pad 3: GND -> Net-(J9-Pin_3)
- R100 pad 2: Net-(J30-Pin_2) -> Net-(J30-Pin_3)
- R102 pad 2: Net-(J31-Pin_2) -> Net-(J31-Pin_3)
- R104 pad 1: Net-(U33-+) -> Net-(U40-+)
- R104 pad 2: Net-(J32-Pin_2) -> Net-(U16--)
- R105 pad 1: GND -> Net-(U41-+)
- R105 pad 2: Net-(U33-+) -> Net-(U17--)
- R106 pad 2: Net-(J35-Pin_2) -> Net-(J18-Pin_3)
- R3 pad 1: GND -> Net-(D42-K)
- R3 pad 2: /VSENSE1 -> Net-(J32-Pin_2)
- R6 pad 1: /VSENSE2 -> Net-(U37-+)
- R6 pad 2: Net-(D4-A) -> Net-(U36--)
- R67 pad 2: Net-(J18-Pin_2) -> Net-(J9-Pin_3)
- R68 pad 2: Net-(J19-Pin_2) -> Net-(J19-Pin_3)
- R7 pad 1: GND -> Net-(U39-+)
- R7 pad 2: /VSENSE2 -> Net-(U15--)
- R70 pad 2: Net-(J20-Pin_2) -> Net-(J20-Pin_3)
- R72 pad 2: Net-(J21-Pin_2) -> Net-(J21-Pin_3)
- R74 pad 2: Net-(J22-Pin_2) -> Net-(J22-Pin_3)
- R76 pad 2: Net-(J23-Pin_2) -> Net-(J23-Pin_3)
- R78 pad 2: Net-(J24-Pin_2) -> Net-(J24-Pin_3)
- R80 pad 2: Net-(J25-Pin_2) -> Net-(J25-Pin_3)
- R84 pad 2: Net-(J26-Pin_2) -> Net-(J26-Pin_3)
- R86 pad 2: Net-(J27-Pin_2) -> Net-(J27-Pin_3)
- R88 pad 2: Net-(J28-Pin_2) -> Net-(J28-Pin_3)
- R90 pad 2: Net-(J29-Pin_2) -> Net-(J29-Pin_3)
- R94 pad 2: /NDQ_AI_GND -> GND
- R95 pad 2: /NDQ_AI_GND -> GND
- R98 pad 1: /NDQ_AI_GND -> GND
- R99 pad 1: /NDQ_AI_GND -> GND
- U13 pad 7: /TC0/MISO -> /TC_POCI
- U14 pad 7: /TC1/MISO -> /TC_POCI
- U15 pad 1: /PT0_read -> Net-(U15--)
- U15 pad 4: /PT0_read -> Net-(U15--)
- U15 pad 5: +3.3V -> +10V
- U16 pad 1: /PT1_read -> Net-(U16--)
- U16 pad 4: /PT1_read -> Net-(U16--)
- U16 pad 5: +3.3V -> +10V
- U17 pad 1: /PT2_read -> Net-(U17--)
- U17 pad 4: /PT2_read -> Net-(U17--)
- U17 pad 5: +3.3V -> +10V
- U18 pad 5: +3.3V -> +10V
- U19 pad 7: /TC2/MISO -> /TC_POCI
- U2 pad 24: /420_ext4_r -> /V_SENSE2
- U2 pad 25: unconnected-(U2-PC5-Pad25) -> /V_SENSE3
- U2 pad 26: /PWR0 -> /V_SENSE0
- U2 pad 27: /PWR1 -> /V_SENSE1
- U20 pad 5: +3.3V -> +10V
- U21 pad 5: +3.3V -> +10V
- U22 pad 5: +3.3V -> +10V
- U23 pad 5: +3.3V -> +10V
- U24 pad 5: +3.3V -> +10V
- U25 pad 5: +3.3V -> +10V
- U28 pad 5: +3.3V -> +10V
- U29 pad 5: +3.3V -> +10V
- U31 pad 1: /420_ext2_r -> Net-(U31--)
- U31 pad 4: /420_ext2_r -> Net-(U31--)
- U32 pad 1: /420_ext3_r -> Net-(U32--)
- U32 pad 4: /420_ext3_r -> Net-(U32--)
- U34 pad 1: /420_ext1_r -> Net-(U34--)
- U34 pad 4: /420_ext1_r -> Net-(U34--)
Routing:
- net +10V: track 0.00 -> 71.8 mm, vias 0 -> 1
- net +3.3V: track 0.00 -> 46.3 mm, vias 0 -> 1
- net /E-Match0/PWR: track 0.00 -> 45.2 mm
- net +24V: track 0.00 -> 45.1 mm, vias 0 -> 16
- net Net-(D6-A): track 0.00 -> 19.9 mm
- net Net-(D5-A): track 0.00 -> 19.4 mm
- net Net-(U20--): track 0.00 -> 9.72 mm
- net Net-(U23--): track 0.00 -> 9.72 mm
- net Net-(U28--): track 0.00 -> 9.72 mm
- net Net-(U24--): track 0.00 -> 9.72 mm
- net Net-(U29--): track 0.00 -> 9.72 mm
- net Net-(U22--): track 0.00 -> 9.72 mm
- net Net-(U21--): track 0.00 -> 9.72 mm
- net Net-(U16--): track 0.00 -> 9.72 mm
- net Net-(U17--): track 0.00 -> 9.72 mm
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- added copper zone on B.Cu, net +3.3V
- added copper zone on F.Cu, net Net-(D1-K)
- added copper zone on B.Cu, net Net-(D2-K)
Other:
- board size 3.2 x 15.6 mm -> 270 x 152 mm
- copper layers 2 -> 4
- board text added: "PT0"

Commit message: Updated to add new filtering circuit
Parts:
- added REF**: UCIRP_Logo_2, UCIRP-KiCAD-Lib:UCIRP_Logo_2, F.Cu at (173.5, 117.2)
- moved D15 294.5 mm to (57.5, 72.7)
- moved J8 294.5 mm to (50.3, 53.0)
- moved Q4 294.5 mm to (54.0, 65.2)
- moved R22 294.5 mm to (57.5, 66.3)
- moved R24 294.5 mm to (56.0, 69.4)
- moved R25 294.5 mm to (53.5, 72.0)
- moved U7 294.5 mm to (49.6, 72.8)
- moved C14 294.5 mm to (46.7, 72.3)
- moved D14 294.5 mm to (49.4, 66.9)
- moved R23 294.5 mm to (56.4, 66.3)
- moved D24 294.1 mm to (46.9, 38.9)
- moved D25 294.1 mm to (55.1, 44.7)
- moved J39 294.1 mm to (47.8, 25.1)
- moved Q10 294.1 mm to (51.5, 37.2)
- moved R46 294.1 mm to (55.1, 38.3)
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Routing:
- net +3.3V: track 46.3 -> 95.3 mm
- net +24V: track 45.1 -> 81.9 mm, vias 16 -> 28
- net Net-(D17-K): track 6.72 -> 26.9 mm
- net Net-(D13-K): track 6.72 -> 26.9 mm
- net Net-(D21-K): track 6.72 -> 26.9 mm
- net Net-(D25-K): track 6.72 -> 26.9 mm
- net Net-(D15-K): track 6.72 -> 26.9 mm
- net Net-(D23-K): track 6.72 -> 26.9 mm
- net Net-(D9-K): track 6.72 -> 26.9 mm
- net Net-(D11-K): track 6.72 -> 26.9 mm
- net Net-(D12-A): track 9.25 -> 27.8 mm
- net Net-(D14-A): track 9.25 -> 27.8 mm
- net Net-(D22-A): track 9.25 -> 27.8 mm
- net Net-(D20-A): track 9.25 -> 27.8 mm
- net Net-(D16-A): track 9.25 -> 27.8 mm
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- added copper zone on B.Cu, net +10V
- added copper zone on B.Cu, net +10V_LOAD_CELL
- added copper zone on B.Cu, net +20V
- added copper zone on B.Cu, net +24V
- added copper zone on B.Cu, net Net-(D10-A)
- added copper zone on F.Cu, net Net-(D10-A)
- added copper zone on B.Cu, net Net-(D12-A)
- added copper zone on F.Cu, net Net-(D12-A)
- added copper zone on B.Cu, net Net-(D14-A)
- added copper zone on F.Cu, net Net-(D14-A)
- added copper zone on B.Cu, net Net-(D16-A)
- added copper zone on F.Cu, net Net-(D16-A)
- added copper zone on B.Cu, net Net-(D18-A)
- added copper zone on B.Cu, net Net-(D20-A)
- added copper zone on F.Cu, net Net-(D20-A)
- added copper zone on B.Cu, net Net-(D22-A)
- added copper zone on F.Cu, net Net-(D22-A)
- added copper zone on B.Cu, net Net-(D24-A)
- added copper zone on F.Cu, net Net-(D24-A)
- added copper zone on B.Cu, net Net-(D8-A)
- added copper zone on F.Cu, net Net-(D8-A)
- added copper zone on B.Cu, net Net-(Q10-S)
- added copper zone on B.Cu, net Net-(Q2-S)
- added copper zone on B.Cu, net Net-(Q3-S)
- added copper zone on B.Cu, net Net-(Q4-S)
- added copper zone on B.Cu, net Net-(Q5-S)
- added copper zone on B.Cu, net Net-(Q6-S)
- added copper zone on B.Cu, net Net-(Q7-S)
- added copper zone on B.Cu, net Net-(Q8-S)
- added copper zone on B.Cu, net Net-(Q9-S)
Other:
- board text added: "By: Reza Bagheri Robert Woo David Culciar Daniel He"
- board text added: "UCI Rocket Project Liquids GSE v2.0 12/2025"
- board text removed: "PT0"

Commit message: Subsystem level layout done (prelim)
Parts:
- removed C101, C103, C104, C106, C107, C109, C53, C55, C61, C84, C85, C86: 100nF, Capacitor_SMD:C_0402_1005Metric
- removed C102, C105, C108, C71, C72, C73, C74, C75, C76, C77, C78, C79, C80, C81, C82, C83: ?, Capacitor_SMD:C_0402_1005Metric
- removed D38, D42, D43, D44, D45: BZT52C3V3LP-7, Diode_SMD:D_0402_1005Metric_Pad0.77x0.64mm_HandSolder
- removed J30, J31: 420Sensor, 0UCIRP-KiCAD-Lib:GX-12 3 pin
- removed R100, R108, R132, R134: 500R, Resistor_SMD:R_0402_1005Metric
- removed R126, R127, R128, R129, R131, R133, R135: 0R, Resistor_SMD:R_0402_1005Metric
- removed U31, U36, U38, U40, U41, U42, U43, U44, U45, U46, U47, U48, U49, U50, U51, U52, U53, U55, U56, U57, U58, U59: ~, Package_TO_SOT_SMD:SOT-23-5
- added C100: 10nF, Capacitor_SMD:C_0603_1608Metric, B.Cu at (31.0, 132.1)
- added C110: 10nF, Capacitor_SMD:C_0603_1608Metric, B.Cu at (91.7, 132.1)
- added C111: 10nF, Capacitor_SMD:C_0603_1608Metric, B.Cu at (51.2, 111.0)
- added C112: 10nF, Capacitor_SMD:C_0603_1608Metric, B.Cu at (71.5, 153.1)
- added C113: 10nF, Capacitor_SMD:C_0603_1608Metric, B.Cu at (51.2, 132.1)
- added C114: 10nF, Capacitor_SMD:C_0603_1608Metric, B.Cu at (51.2, 153.1)
- added C115: 10nF, Capacitor_SMD:C_0603_1608Metric, B.Cu at (29.6, 111.0)
- added C116: 10nF, Capacitor_SMD:C_0603_1608Metric, B.Cu at (71.5, 132.1)
- added C117: 10nF, Capacitor_SMD:C_0603_1608Metric, B.Cu at (31.0, 153.1)
- added C118: 10nF, Capacitor_SMD:C_0603_1608Metric, B.Cu at (91.7, 111.0)
- added C56: 10nF, Capacitor_SMD:C_0603_1608Metric, B.Cu at (91.6, 151.4)
- added C99: 10nF, Capacitor_SMD:C_0603_1608Metric, B.Cu at (71.5, 111.0)
- added D41: BZV55-B5V1, Diode_SMD:D_MiniMELF, B.Cu at (129.0, 115.2)
- added D46: BZV55-B5V1, Diode_SMD:D_MiniMELF, B.Cu at (108.3, 135.8)
- added D47: BZV55-B5V1, Diode_SMD:D_MiniMELF, B.Cu at (128.6, 154.9)
- added R146: 11K, Resistor_SMD:R_0603_1608Metric, B.Cu at (91.6, 148.7)
- added R147: 11K, Resistor_SMD:R_0603_1608Metric, B.Cu at (71.5, 108.2)
- added R148: 11K, Resistor_SMD:R_0603_1608Metric, B.Cu at (31.0, 129.3)
- added R149: 11K, Resistor_SMD:R_0603_1608Metric, B.Cu at (91.7, 129.3)
- added R150: 11K, Resistor_SMD:R_0603_1608Metric, B.Cu at (51.2, 108.2)
- added R151: 11K, Resistor_SMD:R_0603_1608Metric, B.Cu at (71.5, 150.4)
- added R152: 11K, Resistor_SMD:R_0603_1608Metric, B.Cu at (51.2, 129.3)
- added R153: 11K, Resistor_SMD:R_0603_1608Metric, B.Cu at (51.2, 150.4)
- added R154: 11K, Resistor_SMD:R_0603_1608Metric, B.Cu at (29.6, 108.2)
- added R155: 11K, Resistor_SMD:R_0603_1608Metric, B.Cu at (71.5, 129.3)
- added R156: 11K, Resistor_SMD:R_0603_1608Metric, B.Cu at (31.0, 150.4)
- added R157: 11K, Resistor_SMD:R_0603_1608Metric, B.Cu at (91.7, 108.2)
- added R158: 11K, Resistor_SMD:R_0603_1608Metric, B.Cu at (93.6, 148.7)
- added R159: 11K, Resistor_SMD:R_0603_1608Metric, B.Cu at (73.5, 108.2)
- added R160: 11K, Resistor_SMD:R_0603_1608Metric, B.Cu at (33.0, 129.3)
- added R161: 11K, Resistor_SMD:R_0603_1608Metric, B.Cu at (93.7, 129.3)
- added R162: 11K, Resistor_SMD:R_0603_1608Metric, B.Cu at (53.2, 108.2)
- added R163: 11K, Resistor_SMD:R_0603_1608Metric, B.Cu at (73.5, 150.4)
- added R164: 11K, Resistor_SMD:R_0603_1608Metric, B.Cu at (53.2, 129.3)
- added R165: 11K, Resistor_SMD:R_0603_1608Metric, B.Cu at (53.2, 150.4)
- added R166: 11K, Resistor_SMD:R_0603_1608Metric, B.Cu at (31.6, 108.2)
- added R167: 11K, Resistor_SMD:R_0603_1608Metric, B.Cu at (73.5, 129.3)
- added R168: 11K, Resistor_SMD:R_0603_1608Metric, B.Cu at (33.0, 150.4)
- added R169: 11K, Resistor_SMD:R_0603_1608Metric, B.Cu at (93.7, 108.2)
- added R2: 100K, Resistor_SMD:R_0603_1608Metric, B.Cu at (196.8, 75.0)
- added U33: ~, Package_TO_SOT_SMD:SOT-89-3, B.Cu at (247.8, 113.5)
- C10, C12, C13, C14, C16, C17, C18, C19, C2, C20, C21, C22, C23, C24, C25, C3, C32, C33, C4, C44, C5, C6, C63, C64, C65, C66, C67, C68, C7, C8, C87, C88, C89, C9, C90, C91, C92, C93, C94, C95, C96, C97, C98: footprint Capacitor_SMD:C_0402_1005Metric -> Capacitor_SMD:C_0603_1608Metric
- C11, C45, C46, C47, C48, C57: footprint Capacitor_SMD:C_1206_3216Metric -> Capacitor_SMD:C_0603_1608Metric
- C26, C27: footprint Capacitor_SMD:C_1206_3216Metric -> Capacitor_SMD:C_0603_1608Metric; moved to B.Cu
- C28, C29, C30, C31, C34, C35, C36, C37, C38, C39, C40, C41: value 100nF -> 22nF; footprint Capacitor_SMD:C_0402_1005Metric -> Capacitor_SMD:C_0603_1608Metric
- C50: value 0.33uF -> 100nF; footprint Capacitor_SMD:C_1206_3216Metric -> Capacitor_SMD:C_0603_1608Metric
- C51: value 0.1uF -> 100nF; footprint Capacitor_SMD:C_1206_3216Metric -> Capacitor_SMD:C_0603_1608Metric
- C58, C60: footprint Capacitor_SMD:C_0402_1005Metric -> Capacitor_SMD:C_0603_1608Metric; moved to B.Cu
- C59: value ? -> 100nF; footprint Capacitor_SMD:C_0402_1005Metric -> Capacitor_SMD:C_0603_1608Metric; moved to B.Cu
- C69: value ? -> 0.33uF; footprint Capacitor_SMD:C_0402_1005Metric -> Capacitor_SMD:C_0603_1608Metric
- C70: value ? -> 0.1uF; footprint Capacitor_SMD:C_0402_1005Metric -> Capacitor_SMD:C_0603_1608Metric
- D26, D27, D28, D29, D30, D31, D32, D33, D34, D35, D36, D37: value BZT52H -> BZV55-B5V1; footprint Diode_SMD:D_SOD-123F -> Diode_SMD:D_MiniMELF
- D39, D40: value BZT52C3V3LP-7 -> BZV55-B5V1; footprint Diode_SMD:D_0402_1005Metric_Pad0.77x0.64mm_HandSolder -> Diode_SMD:D_MiniMELF; moved to B.Cu
- J18: value 420Sensor -> POT
- Q11, Q12, Q13, Q14, U32, U34, U37: moved to B.Cu
- R1, R10, R109, R11, R110, R111, R112, R113, R114, R115, R116, R117, R12, R13, R15, R16, R17, R18, R19, R21, R22, R23, R25, R26, R27, R29, R30, R31, R32, R34, R35, R37, R38, R39, R4, R41, R42, R43, R45, R46, R47, R49, R5, R62, R63, R64, R65, R8, R82, R83, R9, R94, R95, R98, R99: footprint Resistor_SMD:R_0402_1005Metric -> Resistor_SMD:R_0603_1608Metric
- R101: value 165R -> 5K; footprint Resistor_SMD:R_0402_1005Metric -> Resistor_SMD:R_0603_1608Metric; moved to B.Cu
- R102, R106: value 500R -> 10K; footprint Resistor_SMD:R_0402_1005Metric -> Resistor_SMD:R_0603_1608Metric; moved to B.Cu
- R103, R107: value 165R -> 1K; footprint Resistor_SMD:R_0402_1005Metric -> Resistor_SMD:R_0603_1608Metric; moved to B.Cu
- R104: value 0R -> 15K; footprint Resistor_SMD:R_0402_1005Metric -> Resistor_SMD:R_0603_1608Metric
- R105, R118, R121, R124: value 0R -> 5K; footprint Resistor_SMD:R_0402_1005Metric -> Resistor_SMD:R_0603_1608Metric
- R119, R122, R125: value 0R -> 10K; footprint Resistor_SMD:R_0402_1005Metric -> Resistor_SMD:R_0603_1608Metric
- R120, R123: value 0R -> 1K; footprint Resistor_SMD:R_0402_1005Metric -> Resistor_SMD:R_0603_1608Metric
- R14, R20, R24, R28, R33, R36, R40, R44, R48: footprint Resistor_SMD:R_2512_6332Metric -> Resistor_SMD:R_0603_1608Metric
- R3: value 500R -> 15K; footprint Resistor_SMD:R_0402_1005Metric -> Resistor_SMD:R_0603_1608Metric; moved to B.Cu
- R50, R51, R52, R53, R54, R55, R56, R57, R58, R59, R60, R61: footprint Resistor_SMD:R_0402_1005Metric -> Resistor_SMD:R_0603_1608Metric; moved to B.Cu
- R6: value 0R -> 1K; footprint Resistor_SMD:R_0402_1005Metric -> Resistor_SMD:R_0603_1608Metric; moved to B.Cu
- R66, R69, R71, R73, R75, R77, R79, R81, R85, R87, R89, R91: value 500R -> 200R; footprint Resistor_SMD:R_0402_1005Metric -> Resistor_SMD:R_0603_1608Metric
- R67, R68, R70, R72, R74, R76, R78, R80, R84, R86, R88, R90: value 500R -> 50R; footprint Resistor_SMD:R_0402_1005Metric -> Resistor_SMD:R_0603_1608Metric
- R7: value 0R -> 100K; footprint Resistor_SMD:R_0402_1005Metric -> Resistor_SMD:R_0603_1608Metric
- U35: footprint Package_TO_SOT_SMD:TO-252-2 -> Package_TO_SOT_SMD:SOT-23-5
- moved C70 182.0 mm to (253.0, 115.1), turned to 0 degrees
- moved C69 166.6 mm to (253.0, 111.9), turned to 180 degrees
- moved R104 127.9 mm to (199.4, 96.2), turned to 180 degrees
- moved R3 122.0 mm to (199.4, 74.2), turned to 180 degrees
- moved R7 118.6 mm to (196.8, 95.2)
- moved C51 112.8 mm to (115.3, 154.0), turned to 90 degrees
- moved C50 108.4 mm to (115.3, 113.8), turned to 90 degrees
- moved R123 106.7 mm to (131.1, 150.4), turned to -90 degrees
- moved R125 103.5 mm to (135.3, 156.9), turned to 180 degrees
- moved R119 83.9 mm to (135.8, 117.2), turned to 180 degrees
- moved R105 83.7 mm to (111.8, 156.9), turned to 180 degrees
- moved U35 81.8 mm to (132.8, 114.3), turned to 0 degrees
- moved R122 64.8 mm to (115.0, 137.8), turned to 180 degrees
- moved R124 64.6 mm to (132.1, 156.9), turned to 180 degrees
- moved D40 60.9 mm to (108.3, 154.9), turned to -90 degrees
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Connections:
- C28 pad 1: +10V -> /PT0_read
- C28 pad 2: GND -> Net-(C28-Pad2)
- C29 pad 1: +10V -> /PT1_read
- C29 pad 2: GND -> Net-(C29-Pad2)
- C30 pad 1: +10V -> /PT2_read
- C30 pad 2: GND -> Net-(C30-Pad2)
- C31 pad 1: +10V -> /PT3_read
- C31 pad 2: GND -> Net-(C31-Pad2)
- C34 pad 1: +10V -> /PT4_read
- C34 pad 2: GND -> Net-(C34-Pad2)
- C35 pad 1: +10V -> /PT5_read
- C35 pad 2: GND -> Net-(C35-Pad2)
- C36 pad 1: +10V -> /PT6_read
- C36 pad 2: GND -> Net-(C36-Pad2)
- C37 pad 1: +10V -> /PT7_read
- C37 pad 2: GND -> Net-(C37-Pad2)
- C38 pad 1: +10V -> /PT8_read
- C38 pad 2: GND -> Net-(C38-Pad2)
- C39 pad 1: +10V -> /PT9_read
- C39 pad 2: GND -> Net-(C39-Pad2)
- C40 pad 1: +10V -> /PT10_read
- C40 pad 2: GND -> Net-(C40-Pad2)
- C41 pad 1: +10V -> /PT11_read
- C41 pad 2: GND -> Net-(C41-Pad2)
- C50 pad 1: GND -> +5V
- C50 pad 2: +24V -> GND
- C51 pad 1: +10V_LOAD_CELL -> +5V
- C58 pad 1: +3.3V -> +5V
- C59 pad 1: Net-(U37-+) -> +5V
- C60 pad 1: +3.3V -> +5V
- C69 pad 1: Net-(U39-+) -> GND
- C69 pad 2: GND -> +24V
- C70 pad 1: Net-(U40-+) -> +5V
- C87 pad 1: +10V -> +5V
- C88 pad 1: +10V -> +5V
- C89 pad 1: +10V -> +5V
- C90 pad 1: +10V -> +5V
- C91 pad 1: +10V -> +5V
- C92 pad 1: +10V -> +5V
- C93 pad 1: +10V -> +5V
- C94 pad 1: +10V -> +5V
- C95 pad 1: +10V -> +5V
- C96 pad 1: +10V -> +5V
- C97 pad 1: +10V -> +5V
- C98 pad 1: +10V -> +5V
- GX-1 pad 2: +10V_LOAD_CELL -> +10V
- GX-2 pad 2: +10V_LOAD_CELL -> +10V
- J18 pad 1: +20V -> +5V
- J18 pad 2: unconnected-(J18-Pin_2-Pad2) -> Net-(J18-Pin_2)
- J18 pad 3: Net-(J18-Pin_3) -> GND
- J32 pad 1: +3.3V -> +5V
- J36 pad 1: +3.3V -> +5V
- J37 pad 1: +3.3V -> +5V
- J38 pad 1: +3.3V -> +5V
- R101 pad 1: GND -> /V_SENSE4
- R101 pad 2: Net-(D39-K) -> Net-(U32--)
- R102 pad 1: Net-(D40-K) -> GND
- R102 pad 2: Net-(J31-Pin_3) -> /V_SENSE4
- R103 pad 1: GND -> Net-(J32-Pin_2)
- R104 pad 1: Net-(U40-+) -> GND
- R104 pad 2: Net-(U16--) -> /PWR1
- R105 pad 1: Net-(U41-+) -> /V_SENSE1
- R105 pad 2: Net-(U17--) -> Net-(U34--)
- R106 pad 1: Net-(D38-K) -> GND
- R106 pad 2: Net-(J18-Pin_3) -> /V_SENSE1
- R107 pad 1: GND -> Net-(J36-Pin_2)
- R107 pad 2: Net-(D38-K) -> Net-(D41-K)
- R118 pad 1: Net-(U42-+) -> /V_SENSE0
- R118 pad 2: Net-(U18--) -> Net-(U35--)
- R119 pad 1: Net-(U43-+) -> GND
- R119 pad 2: Net-(U20--) -> /V_SENSE0
- R120 pad 1: Net-(U44-+) -> Net-(J37-Pin_2)
- R120 pad 2: Net-(U21--) -> Net-(D46-K)
- R121 pad 1: Net-(U45-+) -> /V_SENSE2
- R121 pad 2: Net-(U22--) -> Net-(U37--)
- R122 pad 1: Net-(U46-+) -> GND
- R122 pad 2: Net-(U23--) -> /V_SENSE2
- R123 pad 1: Net-(U47-+) -> Net-(J38-Pin_2)
- R123 pad 2: Net-(U24--) -> Net-(D47-K)
- R124 pad 1: Net-(U48-+) -> /V_SENSE3
- R124 pad 2: Net-(U25--) -> Net-(U39--)
- R125 pad 1: Net-(U49-+) -> GND
- R125 pad 2: Net-(U28--) -> /V_SENSE3
- R3 pad 1: Net-(D42-K) -> GND
- R3 pad 2: Net-(J32-Pin_2) -> /PWR0
- R6 pad 1: Net-(U37-+) -> Net-(J18-Pin_2)
- R6 pad 2: Net-(U36--) -> Net-(D39-K)
- R7 pad 1: Net-(U39-+) -> /PWR1
- R7 pad 2: Net-(U15--) -> Net-(D4-A)
- U15 pad 1: Net-(U15--) -> /PT0_read
- U15 pad 3: Net-(D26-K) -> Net-(U15-+)
- U15 pad 4: Net-(U15--) -> /PT0_read
- U15 pad 5: +10V -> +5V
- U16 pad 1: Net-(U16--) -> /PT1_read
- U16 pad 3: Net-(D27-K) -> Net-(U16-+)
- U16 pad 4: Net-(U16--) -> /PT1_read
- U16 pad 5: +10V -> +5V
- U17 pad 1: Net-(U17--) -> /PT2_read
- U17 pad 3: Net-(D28-K) -> Net-(U17-+)
- U17 pad 4: Net-(U17--) -> /PT2_read
- U17 pad 5: +10V -> +5V
- U18 pad 1: Net-(U18--) -> /PT3_read
- U18 pad 3: Net-(D29-K) -> Net-(U18-+)
- U18 pad 4: Net-(U18--) -> /PT3_read
- U18 pad 5: +10V -> +5V
- U2 pad 21: /420_ext1_r -> /V_SENSE0
- U2 pad 22: /420_ext2_r -> /V_SENSE1
- U2 pad 23: /420_ext3_r -> /V_SENSE2
- U2 pad 24: /V_SENSE2 -> /V_SENSE3
- U2 pad 25: /V_SENSE3 -> /V_SENSE4
- U2 pad 26: /V_SENSE0 -> /PWR0
- U2 pad 27: /V_SENSE1 -> /PWR1
- U20 pad 1: Net-(U20--) -> /PT4_read
- U20 pad 3: Net-(D30-K) -> Net-(U20-+)
- U20 pad 4: Net-(U20--) -> /PT4_read
- U20 pad 5: +10V -> +5V
- U21 pad 1: Net-(U21--) -> /PT5_read
- U21 pad 3: Net-(D31-K) -> Net-(U21-+)
- U21 pad 4: Net-(U21--) -> /PT5_read
- U21 pad 5: +10V -> +5V
- U22 pad 1: Net-(U22--) -> /PT6_read
- U22 pad 3: Net-(D32-K) -> Net-(U22-+)
- U22 pad 4: Net-(U22--) -> /PT6_read
- U22 pad 5: +10V -> +5V
- U23 pad 1: Net-(U23--) -> /PT7_read
- U23 pad 3: Net-(D33-K) -> Net-(U23-+)
- U23 pad 4: Net-(U23--) -> /PT7_read
- U23 pad 5: +10V -> +5V
- U24 pad 1: Net-(U24--) -> /PT8_read
- U24 pad 3: Net-(D34-K) -> Net-(U24-+)
- U24 pad 4: Net-(U24--) -> /PT8_read
- U24 pad 5: +10V -> +5V
- U25 pad 1: Net-(U25--) -> /PT9_read
- U25 pad 3: Net-(D35-K) -> Net-(U25-+)
- U25 pad 4: Net-(U25--) -> /PT9_read
- U25 pad 5: +10V -> +5V
- U28 pad 1: Net-(U28--) -> /PT10_read
- U28 pad 3: Net-(D36-K) -> Net-(U28-+)
- U28 pad 4: Net-(U28--) -> /PT10_read
- U28 pad 5: +10V -> +5V
- U29 pad 1: Net-(U29--) -> /PT11_read
- U29 pad 3: Net-(D37-K) -> Net-(U29-+)
- U29 pad 4: Net-(U29--) -> /PT11_read
- U29 pad 5: +10V -> +5V
- U32 pad 3: Net-(D40-K) -> Net-(D39-K)
- U32 pad 5: +3.3V -> +5V
- U34 pad 3: Net-(D38-K) -> Net-(D40-K)
- U34 pad 5: +3.3V -> +5V
- U35 pad 1: +24V -> Net-(U35--)
- U35 pad 3: +10V_LOAD_CELL -> Net-(D41-K)
- U37 pad 1: /V_SENSE1 -> Net-(U37--)
- U37 pad 3: Net-(U37-+) -> Net-(D46-K)
- U37 pad 4: /V_SENSE1 -> Net-(U37--)
- U37 pad 5: +3.3V -> +5V
- U39 pad 1: /PT0_read -> Net-(U39--)
- U39 pad 3: Net-(U39-+) -> Net-(D47-K)
- U39 pad 4: /PT0_read -> Net-(U39--)
- U39 pad 5: +10V -> +5V
Routing:
- net +10V: track 69.0 -> 0.00 mm
- net +24V: track 81.9 -> 36.6 mm, vias 28 -> 162
- net +5V: track 0.00 -> 34.3 mm, vias 0 -> 17
- net +3.3V: track 95.3 -> 66.0 mm, vias 1 -> 0
- net Net-(D22-A): track 27.8 -> 0.00 mm
- net Net-(D12-A): track 27.8 -> 0.00 mm
- net Net-(D8-A): track 27.8 -> 0.00 mm
- net Net-(D14-A): track 27.8 -> 0.00 mm
- net Net-(D10-A): track 27.8 -> 0.00 mm
- net Net-(D20-A): track 27.8 -> 0.00 mm
- net Net-(D24-A): track 27.8 -> 0.00 mm
- net Net-(D16-A): track 27.8 -> 0.00 mm
- net Net-(D17-K): track 26.9 -> 6.23 mm
- net Net-(D13-K): track 26.9 -> 6.23 mm
- net Net-(D21-K): track 26.9 -> 6.23 mm
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- added copper zone on B.Cu, net +5V
- added copper zone on B.Cu, net Net-(Q11-D)
- added copper zone on B.Cu, net Net-(Q13-D)
- removed copper zone on B.Cu, net +10V_LOAD_CELL
- removed copper zone on F.Cu, net Net-(D10-A)
- removed copper zone on F.Cu, net Net-(D12-A)
- removed copper zone on F.Cu, net Net-(D14-A)
- removed copper zone on F.Cu, net Net-(D16-A)
- removed copper zone on F.Cu, net Net-(D20-A)
- removed copper zone on F.Cu, net Net-(D22-A)
- removed copper zone on F.Cu, net Net-(D24-A)
- removed copper zone on F.Cu, net Net-(D8-A)

Commit message: Good progress on full system layout.
Parts:
- C42, C52: value 100nF -> 33nF
- F1: moved to F.Cu
- moved C100 286.8 mm to (317.8, 131.0)
- moved C110 286.8 mm to (378.5, 131.0)
- moved C111 286.8 mm to (338.0, 109.9)
- moved C112 286.8 mm to (358.2, 152.0)
- moved C113 286.8 mm to (338.0, 131.0)
- moved C114 286.8 mm to (338.0, 152.0)
- moved C115 286.8 mm to (316.4, 109.9)
- moved C116 286.8 mm to (358.2, 131.0)
- moved C117 286.8 mm to (317.8, 152.0)
- moved C118 286.8 mm to (378.5, 109.9)
- moved C28 286.8 mm to (382.1, 149.3)
- moved C29 286.8 mm to (362.0, 108.9)
- moved C30 286.8 mm to (321.5, 130.0)
- moved C31 286.8 mm to (382.2, 130.0)
- moved C34 286.8 mm to (341.8, 108.9)
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Connections:
- U2 pad 41: /TC0_~{CS} -> /TC2_~{CS}
- U2 pad 50: /TC2_~{CS} -> /TC0_~{CS}
Routing:
- net /TC_POCI: track 0.00 -> 72.2 mm
- net /TC_SCK: track 0.00 -> 68.3 mm
- net /ETH_CTS: track 0.00 -> 52.0 mm
- net /ETH_RX: track 0.00 -> 51.8 mm
- net /ETH_TX: track 0.00 -> 49.6 mm
- net /ETH_RTS: track 0.00 -> 49.0 mm
- net /ETH_~{RST}: track 0.00 -> 47.3 mm
- net /MCU_~{RST}: track 1.82 -> 44.8 mm, vias 0 -> 2
- net +24V: track 36.6 -> 12.8 mm, vias 162 -> 3
- net /TC0_~{CS}: track 5.24 -> 26.5 mm
- net /TC2_~{CS}: track 5.24 -> 26.2 mm
- net /TC1_~{CS}: track 2.62 -> 17.8 mm, vias 0 -> 2
- net /MCU_SWCLK: track 0.00 -> 13.1 mm
- net /MCU_SWDIO: track 0.00 -> 10.3 mm
- net +3.3V: vias 0 -> 50
- added copper zone on In2.Cu, net +24V
