File: ematch.kicad_sch (KiCad schematic)
At the start: 10 parts, among them J14 E-MATCH, Q11 DMG3402L, Q12 DMG3402L

Commit message: Added LC filter for power filtering
Parts:
- J14: footprint TerminalBlock:TerminalBlock_bornier-2_P5.08mm -> TerminalBlock_MetzConnect:TerminalBlock_MetzConnect_Type055_RT01502HDWU_1x02_P5.00mm_Horizontal
Changed lines of the file:
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@@
 			)
 		)
-		(property "Footprint" "TerminalBlock:TerminalBlock_bornier-2_P5.08mm"
+		(property "Footprint" "TerminalBlock_MetzConnect:TerminalBlock_MetzConnect_Type055_RT01502HDWU_1x02_P5.00mm_Horizontal"
 			(at 168.91 77.47 0)
 			(effects

Commit message: Subsystem level layout done (prelim)
Parts:
- C26: footprint Capacitor_SMD:C_1206_3216Metric -> Capacitor_SMD:C_0603_1608Metric
- R50, R51, R52, R53, R54, R55: footprint Resistor_SMD:R_0402_1005Metric -> Resistor_SMD:R_0603_1608Metric
Changed lines of the file:
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@@
 			)
 		)
-		(property "Footprint" "Resistor_SMD:R_0402_1005Metric"
+		(property "Footprint" "Resistor_SMD:R_0603_1608Metric"
 			(at 194.31 97.79 0)
 			(effects
@@
 			)
 		)
-		(property "Footprint" "Resistor_SMD:R_0402_1005Metric"
+		(property "Footprint" "Resistor_SMD:R_0603_1608Metric"
 			(at 209.55 74.93 0)
 			(effects
@@
 			)
 		)
-		(property "Footprint" "Resistor_SMD:R_0402_1005Metric"
+		(property "Footprint" "Resistor_SMD:R_0603_1608Metric"
 			(at 161.29 86.36 0)
 			(effects
@@
 			)
 		)
-		(property "Footprint" "Capacitor_SMD:C_1206_3216Metric"
+		(property "Footprint" "Capacitor_SMD:C_0603_1608Metric"
 			(at 146.05 82.55 0)
 			(effects
@@
 			)
 		)
-		(property "Footprint" "Resistor_SMD:R_0402_1005Metric"
+		(property "Footprint" "Resistor_SMD:R_0603_1608Metric"
 			(at 146.05 109.22 0)
 			(effects
@@
 			)
 		)
-		(property "Footprint" "Resistor_SMD:R_0402_1005Metric"
+		(property "Footprint" "Resistor_SMD:R_0603_1608Metric"
 			(at 189.23 92.71 0)
 			(effects
@@
 			)
 		)
-		(property "Footprint" "Resistor_SMD:R_0402_1005Metric"
+		(property "Footprint" "Resistor_SMD:R_0603_1608Metric"
 			(at 151.13 104.14 0)
 			(effects

Commit message: GSE v2.1: Updates for DSUB connectors for schematic only done. Layout needs a ton of work
Parts:
- renumbered C26 to C50, J14 to J17, R50 to R72, R51 to R73, R55 to R74, R52 to R75, R53 to R76, R54 to R77
Changed lines of the file:
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@@
 		(dnp no)
 		(fields_autoplaced yes)
-		(property "Reference" "R53"
+		(property "Reference" "R76"
 			(at 196.85 96.52 0)
 			(effects
@@
 			(project "gse2-hardware"
 				(path "/1eb2a3ff-e0fd-4343-8dba-716780a4d459/136c0e1f-4187-47ac-b6b8-3afab399b121"
-					(reference "R53")
-					(unit 1)
-				)
-				(path "/1eb2a3ff-e0fd-4343-8dba-716780a4d459/63f6a9d7-cf1d-42e0-8083-4ad4fb9a9beb"
-					(reference "R60")
-					(unit 1)
-				)
-			)
-		)
-	)
-	(symbol
+					(reference "R76")
+					(unit 1)
+				)
+				(path "/1eb2a3ff-e0fd-4343-8dba-716780a4d459/63f6a9d7-cf1d-42e0-8083-4ad4fb9a9beb"
+					(reference "R82")
+					(unit 1)
+				)
+			)
+		)
+	)
+	(symbol
+		(lib_name "GND_3")
 		(lib_id "power:GND")
 		(at 146.05 111.76 0)
@@
 		(on_board yes)
 		(dnp no)
-		(property "Reference" "#PWR0140"
+		(property "Reference" "#PWR0197"
 			(at 146.05 118.11 0)
 			(effects
@@
 			(project "gse2-hardware"
 				(path "/1eb2a3ff-e0fd-4343-8dba-716780a4d459/136c0e1f-4187-47ac-b6b8-3afab399b121"
-					(reference "#PWR0140")
-					(unit 1)
-				)
-				(path "/1eb2a3ff-e0fd-4343-8dba-716780a4d459/63f6a9d7-cf1d-42e0-8083-4ad4fb9a9beb"
-					(reference "#PWR0146")
+					(reference "#PWR0197")
+					(unit 1)
+				)
+				(path "/1eb2a3ff-e0fd-4343-8dba-716780a4d459/63f6a9d7-cf1d-42e0-8083-4ad4fb9a9beb"
+					(reference "#PWR0203")
 					(unit 1)
 				)
@@
 		(dnp no)
 		(fields_autoplaced yes)
-		(property "Reference" "R54"
+		(property "Reference" "R77"
 			(at 212.09 73.66 0)
 			(effects
@@
 			(project "gse2-hardware"
 				(path "/1eb2a3ff-e0fd-4343-8dba-716780a4d459/136c0e1f-4187-47ac-b6b8-3afab399b121"
-					(reference "R54")
-					(unit 1)
-				)
-				(path "/1eb2a3ff-e0fd-4343-8dba-716780a4d459/63f6a9d7-cf1d-42e0-8083-4ad4fb9a9beb"
-					(reference "R61")
+					(reference "R77")
+					(unit 1)
+				)
+				(path "/1eb2a3ff-e0fd-4343-8dba-716780a4d459/63f6a9d7-cf1d-42e0-8083-4ad4fb9a9beb"
+					(reference "R83")
 					(unit 1)
 				)
@@
 		(on_board yes)
 		(dnp no)
-		(property "Reference" "R55"
+		(property "Reference" "R74"
 			(at 157.48 85.09 0)
 			(effects
@@
 			(project "gse2-hardware"
 				(path "/1eb2a3ff-e0fd-4343-8dba-716780a4d459/136c0e1f-4187-47ac-b6b8-3afab399b121"
-					(reference "R55")
-					(unit 1)
-				)
-				(path "/1eb2a3ff-e0fd-4343-8dba-716780a4d459/63f6a9d7-cf1d-42e0-8083-4ad4fb9a9beb"
-					(reference "R58")
+					(reference "R74")
+					(unit 1)
+				)
+				(path "/1eb2a3ff-e0fd-4343-8dba-716780a4d459/63f6a9d7-cf1d-42e0-8083-4ad4fb9a9beb"
+					(reference "R80")
 					(unit 1)
 				)
@@
 		(on_board yes)
 		(dnp no)
-		(property "Reference" "#PWR0143"
+		(property "Reference" "#PWR0200"
 			(at 209.55 76.2 0)
 			(effects
@@
 			(project "gse2-hardware"
 				(path "/1eb2a3ff-e0fd-4343-8dba-716780a4d459/136c0e1f-4187-47ac-b6b8-3afab399b121"
-					(reference "#PWR0143")
-					(unit 1)
-				)
-				(path "/1eb2a3ff-e0fd-4343-8dba-716780a4d459/63f6a9d7-cf1d-42e0-8083-4ad4fb9a9beb"
-					(reference "#PWR0149")
-					(unit 1)
-				)
-			)
-		)
-	)
-	(symbol
+					(reference "#PWR0200")
+					(unit 1)
+				)
+				(path "/1eb2a3ff-e0fd-4343-8dba-716780a4d459/63f6a9d7-cf1d-42e0-8083-4ad4fb9a9beb"
+					(reference "#PWR0206")
+					(unit 1)
+				)
+			)
+		)
+	)
+	(symbol
+		(lib_name "GND_1")
 		(lib_id "power:GND")
 		(at 194.31 100.33 0)
@@
 		(on_board yes)
 		(dnp no)
-		(property "Reference" "#PWR0142"
+		(property "Reference" "#PWR0199"
 			(at 194.31 106.68 0)
 			(effects
@@
 			(project "gse2-hardware"
 				(path "/1eb2a3ff-e0fd-4343-8dba-716780a4d459/136c0e1f-4187-47ac-b6b8-3afab399b121"
-					(reference "#PWR0142")
-					(unit 1)
-				)
-				(path "/1eb2a3ff-e0fd-4343-8dba-716780a4d459/63f6a9d7-cf1d-42e0-8083-4ad4fb9a9beb"
-					(reference "#PWR0148")
-					(unit 1)
-				)
-			)
-		)
-	)
-	(symbol
+					(reference "#PWR0199")
+					(unit 1)
+				)
+				(path "/1eb2a3ff-e0fd-4343-8dba-716780a4d459/63f6a9d7-cf1d-42e0-8083-4ad4fb9a9beb"
+					(reference "#PWR0205")
+					(unit 1)
+				)
+			)
+		)
+	)
+	(symbol
+		(lib_name "GND_2")
 		(lib_id "power:GND")
 		(at 161.29 109.22 0)
@@
 		(on_board yes)
 		(dnp no)
-		(property "Reference" "#PWR0141"
+		(property "Reference" "#PWR0198"
 			(at 161.29 115.57 0)
 			(effects
@@
 			(project "gse2-hardware"
 				(path "/1eb2a3ff-e0fd-4343-8dba-716780a4d459/136c0e1f-4187-47ac-b6b8-3afab399b121"
-					(reference "#PWR0141")
-					(unit 1)
-				)
-				(path "/1eb2a3ff-e0fd-4343-8dba-716780a4d459/63f6a9d7-cf1d-42e0-8083-4ad4fb9a9beb"
-					(reference "#PWR0147")
+					(reference "#PWR0198")
+					(unit 1)
+				)
+				(path "/1eb2a3ff-e0fd-4343-8dba-716780a4d459/63f6a9d7-cf1d-42e0-8083-4ad4fb9a9beb"
+					(reference "#PWR0204")
 					(unit 1)
 				)
@@
 		(on_board yes)
 		(dnp no)
-		(property "Reference" "C26"
+		(property "Reference" "C50"
 			(at 143.51 81.28 0)
 			(effects
@@
 			(project "gse2-hardware"
 				(path "/1eb2a3ff-e0fd-4343-8dba-716780a4d459/136c0e1f-4187-47ac-b6b8-3afab399b121"
-					(reference "C26")
-					(unit 1)
-				)
-				(path "/1eb2a3ff-e0fd-4343-8dba-716780a4d459/63f6a9d7-cf1d-42e0-8083-4ad4fb9a9beb"
-					(reference "C27")
+					(reference "C50")
+					(unit 1)
+				)
+				(path "/1eb2a3ff-e0fd-4343-8dba-716780a4d459/63f6a9d7-cf1d-42e0-8083-4ad4fb9a9beb"
+					(reference "C51")
 					(unit 1)
 				)
@@
 		(on_board yes)
 		(dnp no)
-		(property "Reference" "#PWR0144"
+		(property "Reference" "#PWR0201"
 			(at 209.55 104.14 0)
 			(effects
@@
 			(project "gse2-hardware"
 				(path "/1eb2a3ff-e0fd-4343-8dba-716780a4d459/136c0e1f-4187-47ac-b6b8-3afab399b121"
-					(reference "#PWR0144")
-					(unit 1)
-				)
-				(path "/1eb2a3ff-e0fd-4343-8dba-716780a4d459/63f6a9d7-cf1d-42e0-8083-4ad4fb9a9beb"
-					(reference "#PWR0150")
+					(reference "#PWR0201")
+					(unit 1)
+				)
+				(path "/1eb2a3ff-e0fd-4343-8dba-716780a4d459/63f6a9d7-cf1d-42e0-8083-4ad4fb9a9beb"
+					(reference "#PWR0207")
 					(unit 1)
 				)
@@
 		(on_board yes)
 		(dnp no)
-		(property "Reference" "J14"
+		(property "Reference" "J17"
 			(at 175.26 77.47 0)
 			(effects
@@
 			(project "gse2-hardware"
 				(path "/1eb2a3ff-e0fd-4343-8dba-716780a4d459/136c0e1f-4187-47ac-b6b8-3afab399b121"
-					(reference "J14")
-					(unit 1)
-				)
-				(path "/1eb2a3ff-e0fd-4343-8dba-716780a4d459/63f6a9d7-cf1d-42e0-8083-4ad4fb9a9beb"
-					(reference "J15")
+					(reference "J17")
+					(unit 1)
+				)
+				(path "/1eb2a3ff-e0fd-4343-8dba-716780a4d459/63f6a9d7-cf1d-42e0-8083-4ad4fb9a9beb"
+					(reference "J18")
 					(unit 1)
 				)
@@
 		(dnp no)
 		(fields_autoplaced yes)
-		(property "Reference" "R50"
+		(property "Reference" "R72"
 			(at 148.59 107.95 0)
 			(effects
@@
 			(project "gse2-hardware"
 				(path "/1eb2a3ff-e0fd-4343-8dba-716780a4d459/136c0e1f-4187-47ac-b6b8-3afab399b121"
-					(reference "R50")
-					(unit 1)
-				)
-				(path "/1eb2a3ff-e0fd-4343-8dba-716780a4d459/63f6a9d7-cf1d-42e0-8083-4ad4fb9a9beb"
-					(reference "R56")
+					(reference "R72")
+					(unit 1)
+				)
+				(path "/1eb2a3ff-e0fd-4343-8dba-716780a4d459/63f6a9d7-cf1d-42e0-8083-4ad4fb9a9beb"
+					(reference "R78")
 					(unit 1)
 				)
@@
 		(on_board yes)
 		(dnp no)
-		(property "Reference" "R52"
+		(property "Reference" "R75"
 			(at 189.23 87.63 90)
 			(effects
@@
 			(project "gse2-hardware"
 				(path "/1eb2a3ff-e0fd-4343-8dba-716780a4d459/136c0e1f-4187-47ac-b6b8-3afab399b121"
-					(reference "R52")
-					(unit 1)
-				)
-				(path "/1eb2a3ff-e0fd-4343-8dba-716780a4d459/63f6a9d7-cf1d-42e0-8083-4ad4fb9a9beb"
-					(reference "R59")
+					(reference "R75")
+					(unit 1)
+				)
+				(path "/1eb2a3ff-e0fd-4343-8dba-716780a4d459/63f6a9d7-cf1d-42e0-8083-4ad4fb9a9beb"
+					(reference "R81")
 					(unit 1)
 				)
@@
 		(on_board yes)
 		(dnp no)
-		(property "Reference" "R51"
+		(property "Reference" "R73"
 			(at 151.13 99.06 90)
 			(effects
@@
 			(project "gse2-hardware"
 				(path "/1eb2a3ff-e0fd-4343-8dba-716780a4d459/136c0e1f-4187-47ac-b6b8-3afab399b121"
-					(reference "R51")
-					(unit 1)
-				)
-				(path "/1eb2a3ff-e0fd-4343-8dba-716780a4d459/63f6a9d7-cf1d-42e0-8083-4ad4fb9a9beb"
-					(reference "R57")
+					(reference "R73")
+					(unit 1)
+				)
+				(path "/1eb2a3ff-e0fd-4343-8dba-716780a4d459/63f6a9d7-cf1d-42e0-8083-4ad4fb9a9beb"
+					(reference "R79")
 					(unit 1)
 				)
@@
 	)
 	(symbol
+		(lib_name "GND_4")
 		(lib_id "power:GND")
 		(at 146.05 85.09 0)
@@
 		(on_board yes)
 		(dnp no)
-		(property "Reference" "#PWR0139"
+		(property "Reference" "#PWR0196"
 			(at 146.05 91.44 0)
 			(effects
@@
 			(project "gse2-hardware"
 				(path "/1eb2a3ff-e0fd-4343-8dba-716780a4d459/136c0e1f-4187-47ac-b6b8-3afab399b121"
-					(reference "#PWR0139")
-					(unit 1)
-				)
-				(path "/1eb2a3ff-e0fd-4343-8dba-716780a4d459/63f6a9d7-cf1d-42e0-8083-4ad4fb9a9beb"
-					(reference "#PWR0145")
-					(unit 1)
-				)
+					(reference "#PWR0196")
+					(unit 1)
+				)
+				(path "/1eb2a3ff-e0fd-4343-8dba-716780a4d459/63f6a9d7-cf1d-42e0-8083-4ad4fb9a9beb"
+					(reference "#PWR0202")
+					(unit 1)
+				)

Commit message: GSE v2.1: Done, ready for JLCPCB
Parts:
- renumbered R72 to R75, R73 to R76, R74 to R77, R75 to R78, R76 to R79, R77 to R80
Changed lines of the file:
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@@
 		(dnp no)
 		(fields_autoplaced yes)
-		(property "Reference" "R76"
+		(property "Reference" "R79"
 			(at 196.85 96.52 0)
 			(effects
@@
 			(project "gse2-hardware"
 				(path "/1eb2a3ff-e0fd-4343-8dba-716780a4d459/136c0e1f-4187-47ac-b6b8-3afab399b121"
-					(reference "R76")
-					(unit 1)
-				)
-				(path "/1eb2a3ff-e0fd-4343-8dba-716780a4d459/63f6a9d7-cf1d-42e0-8083-4ad4fb9a9beb"
-					(reference "R82")
+					(reference "R79")
+					(unit 1)
+				)
+				(path "/1eb2a3ff-e0fd-4343-8dba-716780a4d459/63f6a9d7-cf1d-42e0-8083-4ad4fb9a9beb"
+					(reference "R85")
 					(unit 1)
 				)
@@
 		(on_board yes)
 		(dnp no)
-		(property "Reference" "#PWR0290"
+		(property "Reference" "#PWR0191"
 			(at 146.05 118.11 0)
 			(effects
@@
 			(project "gse2-hardware"
 				(path "/1eb2a3ff-e0fd-4343-8dba-716780a4d459/136c0e1f-4187-47ac-b6b8-3afab399b121"
-					(reference "#PWR0290")
-					(unit 1)
-				)
-				(path "/1eb2a3ff-e0fd-4343-8dba-716780a4d459/63f6a9d7-cf1d-42e0-8083-4ad4fb9a9beb"
-					(reference "#PWR0296")
+					(reference "#PWR0191")
+					(unit 1)
+				)
+				(path "/1eb2a3ff-e0fd-4343-8dba-716780a4d459/63f6a9d7-cf1d-42e0-8083-4ad4fb9a9beb"
+					(reference "#PWR0197")
 					(unit 1)
 				)
@@
 		(dnp no)
 		(fields_autoplaced yes)
-		(property "Reference" "R77"
+		(property "Reference" "R80"
 			(at 212.09 73.66 0)
 			(effects
@@
 			(project "gse2-hardware"
 				(path "/1eb2a3ff-e0fd-4343-8dba-716780a4d459/136c0e1f-4187-47ac-b6b8-3afab399b121"
-					(reference "R77")
-					(unit 1)
-				)
-				(path "/1eb2a3ff-e0fd-4343-8dba-716780a4d459/63f6a9d7-cf1d-42e0-8083-4ad4fb9a9beb"
-					(reference "R83")
+					(reference "R80")
+					(unit 1)
+				)
+				(path "/1eb2a3ff-e0fd-4343-8dba-716780a4d459/63f6a9d7-cf1d-42e0-8083-4ad4fb9a9beb"
+					(reference "R86")
 					(unit 1)
 				)
@@
 		(on_board yes)
 		(dnp no)
-		(property "Reference" "R74"
+		(property "Reference" "R77"
 			(at 157.48 85.09 0)
 			(effects
@@
 			(project "gse2-hardware"
 				(path "/1eb2a3ff-e0fd-4343-8dba-716780a4d459/136c0e1f-4187-47ac-b6b8-3afab399b121"
-					(reference "R74")
-					(unit 1)
-				)
-				(path "/1eb2a3ff-e0fd-4343-8dba-716780a4d459/63f6a9d7-cf1d-42e0-8083-4ad4fb9a9beb"
-					(reference "R80")
+					(reference "R77")
+					(unit 1)
+				)
+				(path "/1eb2a3ff-e0fd-4343-8dba-716780a4d459/63f6a9d7-cf1d-42e0-8083-4ad4fb9a9beb"
+					(reference "R83")
 					(unit 1)
 				)
@@
 		(on_board yes)
 		(dnp no)
-		(property "Reference" "#PWR0288"
+		(property "Reference" "#PWR0194"
 			(at 209.55 76.2 0)
 			(effects
@@
 			(project "gse2-hardware"
 				(path "/1eb2a3ff-e0fd-4343-8dba-716780a4d459/136c0e1f-4187-47ac-b6b8-3afab399b121"
-					(reference "#PWR0288")
-					(unit 1)
-				)
-				(path "/1eb2a3ff-e0fd-4343-8dba-716780a4d459/63f6a9d7-cf1d-42e0-8083-4ad4fb9a9beb"
-					(reference "#PWR0294")
+					(reference "#PWR0194")
+					(unit 1)
+				)
+				(path "/1eb2a3ff-e0fd-4343-8dba-716780a4d459/63f6a9d7-cf1d-42e0-8083-4ad4fb9a9beb"
+					(reference "#PWR0200")
 					(unit 1)
 				)
@@
 		(on_board yes)
 		(dnp no)
-		(property "Reference" "#PWR0292"
+		(property "Reference" "#PWR0193"
 			(at 194.31 106.68 0)
 			(effects
@@
 			(project "gse2-hardware"
 				(path "/1eb2a3ff-e0fd-4343-8dba-716780a4d459/136c0e1f-4187-47ac-b6b8-3afab399b121"
-					(reference "#PWR0292")
-					(unit 1)
-				)
-				(path "/1eb2a3ff-e0fd-4343-8dba-716780a4d459/63f6a9d7-cf1d-42e0-8083-4ad4fb9a9beb"
-					(reference "#PWR0298")
+					(reference "#PWR0193")
+					(unit 1)
+				)
+				(path "/1eb2a3ff-e0fd-4343-8dba-716780a4d459/63f6a9d7-cf1d-42e0-8083-4ad4fb9a9beb"
+					(reference "#PWR0199")
 					(unit 1)
 				)
@@
 		(on_board yes)
 		(dnp no)
-		(property "Reference" "#PWR0289"
+		(property "Reference" "#PWR0192"
 			(at 161.29 115.57 0)
 			(effects
@@
 			(project "gse2-hardware"
 				(path "/1eb2a3ff-e0fd-4343-8dba-716780a4d459/136c0e1f-4187-47ac-b6b8-3afab399b121"
-					(reference "#PWR0289")
-					(unit 1)
-				)
-				(path "/1eb2a3ff-e0fd-4343-8dba-716780a4d459/63f6a9d7-cf1d-42e0-8083-4ad4fb9a9beb"
-					(reference "#PWR0295")
+					(reference "#PWR0192")
+					(unit 1)
+				)
+				(path "/1eb2a3ff-e0fd-4343-8dba-716780a4d459/63f6a9d7-cf1d-42e0-8083-4ad4fb9a9beb"
+					(reference "#PWR0198")
 					(unit 1)
 				)
@@
 		(on_board yes)
 		(dnp no)
-		(property "Reference" "#PWR0291"
+		(property "Reference" "#PWR0195"
 			(at 209.55 104.14 0)
 			(effects
@@
 			(project "gse2-hardware"
 				(path "/1eb2a3ff-e0fd-4343-8dba-716780a4d459/136c0e1f-4187-47ac-b6b8-3afab399b121"
-					(reference "#PWR0291")
-					(unit 1)
-				)
-				(path "/1eb2a3ff-e0fd-4343-8dba-716780a4d459/63f6a9d7-cf1d-42e0-8083-4ad4fb9a9beb"
-					(reference "#PWR0297")
+					(reference "#PWR0195")
+					(unit 1)
+				)
+				(path "/1eb2a3ff-e0fd-4343-8dba-716780a4d459/63f6a9d7-cf1d-42e0-8083-4ad4fb9a9beb"
+					(reference "#PWR0201")
 					(unit 1)
 				)
@@
 		(dnp no)
 		(fields_autoplaced yes)
-		(property "Reference" "R72"
+		(property "Reference" "R75"
 			(at 148.59 107.95 0)
 			(effects
@@
 			(project "gse2-hardware"
 				(path "/1eb2a3ff-e0fd-4343-8dba-716780a4d459/136c0e1f-4187-47ac-b6b8-3afab399b121"
-					(reference "R72")
-					(unit 1)
-				)
-				(path "/1eb2a3ff-e0fd-4343-8dba-716780a4d459/63f6a9d7-cf1d-42e0-8083-4ad4fb9a9beb"
-					(reference "R78")
+					(reference "R75")
+					(unit 1)
+				)
+				(path "/1eb2a3ff-e0fd-4343-8dba-716780a4d459/63f6a9d7-cf1d-42e0-8083-4ad4fb9a9beb"
+					(reference "R81")
 					(unit 1)
 				)
@@
 		(on_board yes)
 		(dnp no)
-		(property "Reference" "R75"
+		(property "Reference" "R78"
 			(at 189.23 87.63 90)
 			(effects
@@
 			(project "gse2-hardware"
 				(path "/1eb2a3ff-e0fd-4343-8dba-716780a4d459/136c0e1f-4187-47ac-b6b8-3afab399b121"
-					(reference "R75")
-					(unit 1)
-				)
-				(path "/1eb2a3ff-e0fd-4343-8dba-716780a4d459/63f6a9d7-cf1d-42e0-8083-4ad4fb9a9beb"
-					(reference "R81")
+					(reference "R78")
+					(unit 1)
+				)
+				(path "/1eb2a3ff-e0fd-4343-8dba-716780a4d459/63f6a9d7-cf1d-42e0-8083-4ad4fb9a9beb"
+					(reference "R84")
 					(unit 1)
 				)
@@
 		(on_board yes)
 		(dnp no)
-		(property "Reference" "R73"
+		(property "Reference" "R76"
 			(at 151.13 99.06 90)
 			(effects
@@
 			(project "gse2-hardware"
 				(path "/1eb2a3ff-e0fd-4343-8dba-716780a4d459/136c0e1f-4187-47ac-b6b8-3afab399b121"
-					(reference "R73")
-					(unit 1)
-				)
-				(path "/1eb2a3ff-e0fd-4343-8dba-716780a4d459/63f6a9d7-cf1d-42e0-8083-4ad4fb9a9beb"
-					(reference "R79")
+					(reference "R76")
+					(unit 1)
+				)
+				(path "/1eb2a3ff-e0fd-4343-8dba-716780a4d459/63f6a9d7-cf1d-42e0-8083-4ad4fb9a9beb"
+					(reference "R82")
 					(unit 1)
 				)
@@
 		(on_board yes)
 		(dnp no)
-		(property "Reference" "#PWR0287"
+		(property "Reference" "#PWR0190"
 			(at 146.05 91.44 0)
 			(effects
@@
 			(project "gse2-hardware"
 				(path "/1eb2a3ff-e0fd-4343-8dba-716780a4d459/136c0e1f-4187-47ac-b6b8-3afab399b121"
-					(reference "#PWR0287")
-					(unit 1)
-				)
-				(path "/1eb2a3ff-e0fd-4343-8dba-716780a4d459/63f6a9d7-cf1d-42e0-8083-4ad4fb9a9beb"
-					(reference "#PWR0293")
-					(unit 1)
-				)
+					(reference "#PWR0190")
+					(unit 1)
+				)
+				(path "/1eb2a3ff-e0fd-4343-8dba-716780a4d459/63f6a9d7-cf1d-42e0-8083-4ad4fb9a9beb"
+					(reference "#PWR0196")
+					(unit 1)
+				)
