File: gse2-hardware.kicad_sch (KiCad schematic)
At the start: 89 parts, among them J1 PJ-002A, J2 PJ-002A, J3 ARM Cortex Debug, J4 USB-C, J5 DSUB_15pin/VGA Veritical Fema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, J6 ARM, J7 0430451812, Q1 DMG3402L, U1 STM32F105RCT6, U2 AS78L05RTR-E1, U3 USBLC6-2SC6, U4 GC-XPORT, U5 3V3_Buck MP2338GTL-Z, U6 UA78M10CKVURG3, U7 BA78M20FP-E2, U8 MAX11614, Y1 16MHz

Commit message: GSE v2.1: small changes made and typos
Parts:
- J5: value DSUB_15pin/VGA Veritical Female -> DSUB_15pin/VGA Vertical Female
Changed lines of the file:
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@@
 			)
 		)
-		(property "Value" "DSUB_15pin/VGA Veritical  Female"
+		(property "Value" "DSUB_15pin/VGA Vertical  Female"
 			(at 214.376 89.154 0)
 			(effects

Commit message: GSE v2.1: Done, ready for JLCPCB
Parts:
- added U49: L7805, Package_TO_SOT_THT:TO-220-3_Vertical, symbol Regulator_Linear:L7805
- J3: Part # Generic 2x5 1.27mm SMD Pin Header -> X1321WVS-2x05J-C40D53
- renumbered C23 to C22, C25 to C23, C22 to C24, C24 to C25, D56 to D6, D55 to D7, D6 to D8, D54 to D9, R269 to R13, R13 to R14, R14 to R15, R15 to R16, R16 to R17, R17 to R18, R18 to R19, R268 to R20, R19 to R21, R20 to R22, R21 to R23, R22 to R24, R23 to R25, R24 to R26, R25 to R27, R267 to R28, R26 to R29
Connections:
- net +24V: now also U49.1 (IN)
- net +5V: now also U49.3 (OUT)
- net GND: now also U49.2 (GND)
Other:
- removed sheet STM_PT4
- removed sheet STM_PT5
- removed sheet STM_PT6
- removed sheet STM_PT7
- added sheet Loadcell2 (loadcell.kicad_sch)
- added sheet Loadcell3 (loadcell.kicad_sch)
- added sheet Loadcell4 (loadcell.kicad_sch)
- added sheet Loadcell5 (loadcell.kicad_sch)
- note added: "Backup LDO"
- note added: "Currently BA178M20FP-E2 on GSE v2.1 4/8/26"
- moved on the sheet: C12, C15, D6, R13, U2
